Commit message: fix: 그리퍼 RViz TF 표시 및 닫힘 동작 수정
- check_gripper.rviz 파일에서 TF Prefix가 "/"로 남아있어 전체 링크에서
  TF 메시지를 잘못 파싱하려고 하여 로봇팔이 제대로 표시되지 못하던 문제 수정
  (RViz의 좌측 RobotModel Display 항목 중 TF Prefix를 빈 문자열로 변경)
- finger2_joint를 mimic으로 전환, finger1_joint 기준 대칭 동작하도록
  axis 반전
- 손가락 원점을 완전히 열린 위치로 재정의하고 limit upper를 조정해
  그리퍼가 실제로 닫히도록 수정

File: src/arm_description/urdf/arm_gripper.urdf.xacro (robot description, xacro)
@@ -40,17 +40,24 @@
   </inertial>
 </link>
+<!-- Mimic 방식 적용. Joint는 두 개 다 필요. finger1_joint를 기준으로
+  finger2_joint를 mimic joint로 설정
+  finger2_joint의 axis에서 y축을 반대로 설정하여 y축 값이 커지면 중심 반대로 이동하도록 함
+  원점을 그리퍼가 완전히 열린 상태로 지정. 그리퍼 두깨가 0.01이므로 finger1_joint와
+   finger2_joint의 limit upper를 0.025로 설정하여 그리퍼가 닫히도록 함
+  -->
 <joint name="finger1_joint" type="prismatic">
   <parent link="tool0"/>
   <child link="finger1_link"/>
-  <origin xyz="0 0.02 0.05" rpy="0 0 0"/>
-  <axis xyz="0 1 0"/>
-  <limit lower="0.0" upper="0.04" effort="20" velocity="0.1"/>
+  <origin xyz="0 0.03 0.05" rpy="0 0 0"/>
+  <axis xyz="0 -1 0"/>
+  <limit lower="0.0" upper="0.025" effort="20" velocity="0.1"/>
 </joint>
 <joint name="finger2_joint" type="prismatic">
   <parent link="tool0"/>
   <child link="finger2_link"/>
-  <origin xyz="0 -0.02 0.05" rpy="0 0 0"/>
+  <origin xyz="0 -0.03 0.05" rpy="0 0 0"/>
   <axis xyz="0 1 0"/>
-  <limit lower="0.0" upper="0.04" effort="20" velocity="0.1"/>
+  <limit lower="0.0" upper="0.025" effort="20" velocity="0.1"/>
+  <mimic joint="finger1_joint" multiplier="1.0" offset="0.0"/>
 </joint>
 </robot>

Commit message: feat: 그리퍼 전용 액션 컨트롤러, TCP 프레임, 픽업 대상물 추가
- arm_controllers.yaml에 gripper_controller(parallel_gripper_action_controller)
  등록, finger1_joint를 joint_trajectory_controller에서 제외
  (인터페이스 점유 충돌 방지)
- arm_study_bringup.launch.py에 gripper_controller 스포너 추가
- arm_gripper.urdf.xacro에 tcp_link 추가 (tool0 기준 z=0.075,
  손끝 사이 중심 — 그립 목표 좌표 기준점)
- 픽업 대상물(board.sdf)을 새로 생성, CMakeLists.txt에 models
  디렉토리 install 규칙 추가
- board 생성 위치를 create 노드의 -x/-y/-z 인자로 지정
  (ros_gz_sim create -file 옵션으로 생성하면 파일 내 <pose>를
  무시하고 원점에 생성됨)

File: src/arm_description/urdf/arm_gripper.urdf.xacro (robot description, xacro)
@@ -58,3 +58,15 @@
   <mimic joint="finger1_joint" multiplier="1.0" offset="0.0"/>
 </joint>
+<!-- TCP (Tool Center Point) link
+  물체를 잡을 때 사용하는 그리퍼의 중심점에 대한 가상 좌표계이다.
+  TCP link는 tool0 link에서 z축으로 0.075m 떨어진 손가락 끝에 위치하도록 설정.
+  (finger1_joint 원점: tool0 기준 z축으로 0.05, 그리퍼의 길이 0.05m, 따라서 0.05 + 0.05/2 = 0.075m)
+  TCP link는 고정 링크로 설정하여, 그리퍼가 움직이더라도 TCP link는 tool0 link에 고정되도록 함.
+-->
+<link name="tcp_link"/>
+<joint name="tcp_joint" type="fixed">
+  <parent link="tool0"/>
+  <child link="tcp_link"/>
+  <origin xyz="0 0 0.075" rpy="0 0 0"/>
+</joint>
 </robot>

Commit message: fix(description): 그리퍼 개방폭을 50mm 에서 70mm 로 확대
1) 손가락 원점을 중심에서 ±30mm 에서 ±40mm 로 이동. 비전 인식 오차 허용치를 늘임
2) limit upper 도 0.025 에서 0.035 로 변경.
3) 접촉까지 이동량이 늘어나기 때문에 velocity 를 0.1 에서 0.3 으로 상향
  (시각적으로는 빨라진 것으로 보임)

File: src/arm_description/urdf/arm_gripper.urdf.xacro (robot description, xacro)
@@ -41,19 +41,19 @@
   finger2_joint의 axis에서 y축을 반대로 설정하여 y축 값이 커지면 중심 반대로 이동하도록 함
   원점을 그리퍼가 완전히 열린 상태로 지정. 그리퍼 두깨가 0.01이므로 finger1_joint와
-   finger2_joint의 limit upper를 0.025로 설정하여 그리퍼가 닫히도록 함
+   finger2_joint의 limit upper를 0.035로 설정하여 그리퍼가 닫히도록 함
   -->
 <joint name="finger1_joint" type="prismatic">
   <parent link="tool0"/>
   <child link="finger1_link"/>
-  <origin xyz="0 0.03 0.05" rpy="0 0 0"/>
+  <origin xyz="0 0.04 0.05" rpy="0 0 0"/>
   <axis xyz="0 -1 0"/>
-  <limit lower="0.0" upper="0.025" effort="20" velocity="0.1"/>
+  <limit lower="0.0" upper="0.035" effort="20" velocity="0.3"/>
 </joint>
 <joint name="finger2_joint" type="prismatic">
   <parent link="tool0"/>
   <child link="finger2_link"/>
-  <origin xyz="0 -0.03 0.05" rpy="0 0 0"/>
+  <origin xyz="0 -0.04 0.05" rpy="0 0 0"/>
   <axis xyz="0 1 0"/>
-  <limit lower="0.0" upper="0.025" effort="20" velocity="0.1"/>
+  <limit lower="0.0" upper="0.035" effort="20" velocity="0.3"/>
   <mimic joint="finger1_joint" multiplier="1.0" offset="0.0"/>
 </joint>

Commit message: fix(description): ros2_control이 finger2_joint의  mimic 제어를 하지 못하도록 막음.
URDF 의 <mimic> 은 SDF 로 변환되어 물리 엔진의 기어 제약을 만든다. gz_ros2_control 도
같은 태그를 읽어 follower 에 속도 명령을 따로 넣는다.
즉, finger2 joint 에 물리적 제약에 의한 이동과 제어기에 의한 속도 명령이 한 번에 주어진다.
이로 인해, 그리퍼가 닫히지 못하거나, 목표를 넘어서 이동하거나, 시뮬레이션마다 결과가 달라지는
현상이 발생하였다.
그래서 이 둘 중 하나를 동작하지 않도록 할 필요가 있으며 그 방법으로 <ros2_control> 의
joint 태그에 mimic="false" 를 주어서 ros2_control의 제어가 꺼지도록 하였다.
Gazebo의 물리 제약은 그대로 두어 finger2 는 finger1 을 따라가는 mimic 동작은 정상

File: src/arm_description/urdf/arm_gripper.urdf.xacro (robot description, xacro)
@@ -1,5 +1,5 @@
 <?xml version="1.0"?>
 <robot xmlns:xacro="http://wiki.ros.org/xacro">
-<!-- ① 인자 선언: launch나 CLI에서 값을 바꿔 넣을 수 있는 변수 -->
+<!-- 인자 선언: launch나 CLI에서 값을 바꿔 넣을 수 있는 변수 -->
   <xacro:arg name="name"      default="ur5e"/>
   <xacro:arg name="ur_type"   default="ur5e"/>

File: src/arm_description/urdf/gripper_joint_control.xacro (robot description, xacro)
@@ -20,5 +20,5 @@
       </state_interface>
     </joint>
-    <joint name="${tf_prefix}finger2_joint">
+    <joint name="${tf_prefix}finger2_joint" mimic="false">
       <state_interface name="position">
         <param name="initial_value">${initial_positions['finger2_joint']}</param>
